Commit message: big update

File: src/webots_ros2_ugv/resource/ugv_webots.urdf (robot description, URDF)
Before this commit: robot UGV Webots, 5 links, 4 joints
Links:
- link base_link: geometry visual box size=4.84 1.72 1.5
Joints:
- joint base_joint: origin xyz=0 0 0 rpy=0 0 0 -> xyz=1.37 0 0 rpy=0 0 0
