Commit message: failed attempt to make mechanical linkages work

File: src/beetle_description/urdf/beetle.urdf (robot description, URDF)
Before this commit: robot beetle, 2 links, 3 joints
Joints:
- added joint steering_rack1_joint: type prismatic, parent left_steering_coupler_link, child steering_rack1_link, origin xyz=${steering_rack_yoff} 0 ${steering_arm_thickness} rpy=0 0 0, axis 1 0 0, limit lower=-0.050 upper=0.050 effort=1000 velocity=1.0
- added joint steering_rack_joint: type prismatic, parent right_steering_coupler_link, child steering_rack_link, origin xyz=${steering_rack_yoff} 0 ${steering_arm_thickness} rpy=0 0 0, axis 1 0 0, limit lower=-0.050 upper=0.050 effort=1000 velocity=1.0
