Commit message: update urdf

File: beetle_description/urdf/beetle.urdf (robot description, URDF)
Before this commit: robot beetle, 2 links, 5 joints
Joints:
- removed joint steering_rack1_joint

Commit message: fix links masses

File: beetle_description/urdf/beetle.urdf (robot description, URDF)
Before this commit: robot beetle, 2 links, 4 joints
Joints:
- joint steering_rack_joint: limit lower=-0.050 upper=0.050 effort=1000 velocity=1.0 -> lower=-0.050 upper=0.050 effort=30000 velocity=1.0

Commit message: add differential gearbox

File: beetle_description/urdf/beetle.urdf (robot description, URDF)
Before this commit: robot beetle, 2 links, 4 joints
Links:
- added link ring_gear_link; collision cylinder length=${ring_gear_thickness} radius=${ring_gear_radius}; visual cylinder length=${ring_gear_thickness} radius=${ring_gear_radius}
- added link spider_gear_link; collision cylinder length=${spider_gear_thickness} radius=${spider_gear_radius}; visual cylinder length=${spider_gear_thickness} radius=${spider_gear_radius}
Joints:
- added joint ring_gear_joint: type continuous, parent base_link, child ring_gear_link, origin xyz=0 ${ring_gear_yoff} ${rear_axle_zoff} rpy=${-pi/2} 0 0, axis 0 0 1
- added joint spider_gear_joint: type continuous, parent ring_gear_link, child spider_gear_link, origin xyz=0 0 ${ring_gear_yoff} rpy=${-pi/2} 0 0, axis 0 0 1

Commit message: finish mechanical simulation for the robot

File: beetle_description/urdf/beetle.urdf (robot description, URDF)
Before this commit: robot beetle, 4 links, 6 joints
Joints:
- removed joint steering_rack_joint
- added joint steering_slider_joint: type prismatic, parent right_steering_coupler_link, child steering_slider_link, origin xyz=${steering_slider_yoff} 0 ${steering_arm_width} rpy=0 ${-pi/2} 0, axis 0 0 1, limit lower=${-steering_slider_limit} upper=${steering_slider_limit} effort=30000 velocity=1.0
- joint ring_gear_joint: limit (none) -> effort=1000 velocity=${2*pi}

Commit message: add stereo camera to simulation

File: beetle_description/urdf/beetle.urdf (robot description, URDF)
Before this commit: robot beetle, 2 links, 3 joints
Links:
- added link camera, mass 0.1; collision box size=0.1 0.4 0.1; visual box size=0.1 0.4 0.1
- added link camera_depth_frame
- added link camera_rgb_frame
Joints:
- added joint camera_depth_joint: type fixed, parent camera, child camera_depth_frame, origin xyz=0 0 0 rpy=${pi/2} ${pi} ${pi/2}
- added joint camera_joint: type fixed, parent base_link, child camera, origin xyz=1 0 0.75 rpy=0 ${pi/8} 0
- added joint camera_optical_joint: type fixed, parent camera, child camera_rgb_frame, origin xyz=0 0 0 rpy=0 0 0
